File: RC-KAKATA-CONTROL/RC-KAKATA-CONTROL.kicad_sch (KiCad schematic)
At the start: 64 parts, among them J1 Conn_02x20_Socket_DG250T-5.0-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, J10 DB125-2.54-4P-GN, J12 Conn_01x07, J25 Conn_02x20_Socket_DG250T-5.0-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, J6 Raspberry_Pi_2x20_PTH, J8 DB125-2.54-4P-GN, U3 STM32H743IIT6, U5 DB125-2.54-6P-GN, U8 W25Q128JVSIQTR, X1 SMD3225-4, X2 Q13MC3061000300

Commit message: Agregadas conexiones de analogicos Agregadas las conexiones de i2c Agregadas las conexiones de Uart Cambiados algunos detalles de tvs resistencias y cap Recolocados los componenetes de power supply Cambiados los diodos de entrada de la bateria por unos de 5A Cambios menores y mejorada la documentacion Agregada informacion en la serigrafia del PCB
Parts:
- removed D10, D11, D12, D9: PESD3V3L1BA, Diode_SMD_AKL:D_SOD-323_TVS, symbol Diode_TVS_AKL:PESD3V3L1BA
- removed R38, R39: 10K, 4ms_Resistor:R_0603, symbol MG_RESISTOR:RES-0603-10K-1%
- removed U5: DB125-2.54-6P-GN, EasyEDA:CONN-TH_DB125-2.54-6P-GN, symbol EasyEDA:DB125-2.54-6P-GN
- added C51, C52, C53, C54: 100NF, 4ms_Capacitor:C_0603, symbol MG_CAPACITOR:CAP-0603-100NF-16V-X5R
- R20, R21, R22, R23, R24, R25, R26, R27, R28, R29, R30, R31, R32, R33, R34, R35, R36, R37: value 10K -> 22K
Connections:
- net ENC_B_DELANTERO_DER is gone; now on net LS_DELANTERO_DX_180G: J1.7 (Pin_7), R33.2
- net ENC_B_DELANTERO_IZQ is gone; now on net LS_DELANTERO_DX_0G: J1.8 (Pin_8), R32.2
- net ENC_B_MOTOR_1_DER is gone; now on net LS_TRASERO_DX_180G: J1.3 (Pin_3), R37.2
- net ENC_B_MOTOR_1_IZQ is gone; now on net LS_TRASERO_IX_0G: J1.6 (Pin_6), R34.2
- net ENC_B_MOTOR_2_IZQ is gone; now on net LS_TRASERO_IX_180G: J1.5 (Pin_5), R35.2
- net ENC_B_MOTOR_3_IZQ is gone; now on net LS_TRASERO_DX_0G: J1.4 (Pin_4), R36.2
- net ENC_B_TRASERO_DER is gone; now on net LS_DELANTERO_IX_180G: J1.9 (Pin_9), R31.2
- net ENC_B_TRASERO_IZQ is gone; now on net LS_DELANTERO_IX_0G: J1.10 (Pin_10), R30.2
- net ACC_GYR_INT: now also U3.156 (PG13)
- net ACC_GYR_SCL: now also R4.2, U3.17 (PF1)
- net ACC_GYR_SDA: now also R3.2, U3.16 (PF0)
- net ACC_I2C_SCL: now also R1.2, U3.164 (PB6)
- net ACC_I2C_SDA: now also R2.2, U3.165 (PB7)
- net BUTON1: now also U3.131 (PI0)
- net BUTON2: now also U3.132 (PI1)
- net BUTON3: now also U3.133 (PI2)
- net BUTON4: now also U3.134 (PI3)
- net DIR_A_DELANTERO_DER: now also U3.110 (PG6)
- net DIR_A_DELANTERO_IZQ: now also U3.108 (PG4)
- net DIR_A_MOTOR_DER: now also U3.153 (PG10)
- net DIR_A_MOTOR_IZQ: now also U3.112 (PG8)
- net DIR_A_TRASERO_DER: now also U3.106 (PG2)
- net DIR_A_TRASERO_IZQ: now also U3.66 (PG0)
- net DIR_B_DELANTERO_DER: now also U3.111 (PG7)
- net DIR_B_DELANTERO_IZQ: now also U3.109 (PG5)
- net DIR_B_MOTOR_DER: now also U3.154 (PG11)
- net DIR_B_MOTOR_IZQ: now also U3.152 (PG9)
- net DIR_B_TRASERO_DER: now also U3.107 (PG3)
- net DIR_B_TRASERO_IZQ: now also U3.67 (PG1)
- net GND: now also C51.2, C52.2, C53.2, C54.2
- net JOY_DIRA: now also U3.56 (PB0)
- net JOY_DIRB: now also U3.57 (PB1)
- net JOY_PB: now also U3.155 (PG12)
- net UART_RX: now also U3.92 (PB12)
- net UART_TX: now also U3.93 (PB13)
- net LS_TRASERO_IX_180G: now reaches U3.11 (PI9)
- net LS_TRASERO_IX_180G: now also C53.1
- net LS_TRASERO_DX_0G: now reaches U3.12 (PI10)
- net LS_TRASERO_DX_0G: now also C52.1
- net LS_TRASERO_DX_180G: now reaches U3.13 (PI11)
- net LS_TRASERO_DX_180G: now also C51.1
- net LS_DELANTERO_IX_0G: now reaches U3.173 (PI4)
- net LS_DELANTERO_IX_0G: now also C32.1
- net LS_DELANTERO_IX_180G: now reaches U3.174 (PI5)
- net LS_DELANTERO_IX_180G: now also C31.1
- net LS_DELANTERO_DX_0G: now reaches U3.175 (PI6)
- net LS_DELANTERO_DX_0G: now also C30.1
- net LS_DELANTERO_DX_180G: now reaches U3.176 (PI7)
- net LS_DELANTERO_DX_180G: now also C29.1
- net LS_TRASERO_IX_0G: now reaches U3.7 (PI8)
- net LS_TRASERO_IX_0G: now also C54.1
- net ENC_B_MOTOR_2_DER: no longer names the net of J1.2 (Pin_2)
- net ENC_B_MOTOR_3_DER: no longer names the net of J1.1 (Pin_1)
- removed net LSGTD: C29.1, R4.2
- removed net LSGTI: C30.1, R3.2
- removed net LS_GDD: C31.1, R2.2
- removed net LS_GDI: C32.1, R1.2
Other:
- note removed: "LIMIT SW"
- moved on the sheet: C29, C30, C31, C32

Commit message: Colocadas todas las piezas Verificacion de conexiones de los puertos UART - I2C - SPI Realizadas todas las conexiones Verificados los errores
Parts:
- added LED5: LED_0603_Red, LED_SMD_AKL:LED_0603_1608Metric, symbol LED_AKL:LED_0603_Red
- added R18: 300, 4ms_Resistor:R_0603, symbol MG_RESISTOR:RES-0603-10K-1%
- added R19, R38, R39: 10K, 4ms_Resistor:R_0603, symbol MG_RESISTOR:RES-0603-10K-1%
- added R51: 100K, 4ms_Resistor:R_0603, symbol MG_RESISTOR:RES-0603-10K-1%
Connections:
- net +3.3V: now also R19.1, R39.1, R51.1
- net ADC_VBAT1: now also U3.32 (PC0)
- net ADC_VBAT2: now also U3.33 (PC1)
- net GND: now also LED5.1 (K), R38.2
- net JTCK/SWCLK: now also R38.1
- net JTDI: now also J12.4 (Pin_4), R39.2; no longer J12.5 (Pin_5)
- net JTMS/SWDIO: now also R51.2
- net NJTRST: now also J12.5 (Pin_5), R19.2; no longer J12.4 (Pin_4)
- net RF_DATA_IN_TIM: now also U3.1 (PE2)
- net RF_DATA_IN_UART: now also U3.129 (PH14)
- net RF_DATA_TIMER: now also U3.2 (PE3)
- net RF_DATA_UART_TX: now also U3.128 (PH13)
- net RPI_SPI_CLK: now also U3.51 (PA5)
- net RPI_SPI_CS: now also U3.50 (PA4)
- net RPI_SPI_MISO: now also U3.53 (PA7)
- net RPI_SPI_MOSI: now also U3.52 (PA6)
- net RPI_UART2_RX: now also U3.96 (PD8)
- net RPI_UART2_TX: now also U3.97 (PD9)
- net VDDA: now also U3.38 (VREF+)
- net RPI_GPIO_16: now reaches U3.119 (PA8)
- net RPI_GPIO_16: now also J6.36 (GPIO16)
- net RPI_GPIO_17: now reaches U3.120 (PA9)
- net RPI_GPIO_17: now also J6.11 (GPIO17)
- net RPI_GPIO_18: now reaches U3.121 (PA10)
- net RPI_GPIO_18: now also J6.12 (GPIO18/PWM0)
- net RF_DATA_EN: now reaches U3.157 (PG14)
- net RPI_GPIO_SCL: now reaches U3.84 (PH7)
- net RPI_GPIO_SCL: now also J6.5 (SCL/GPIO3)
- net RPI_GPIO_SDA: now reaches U3.85 (PH8)
- net RPI_GPIO_SDA: now also J6.3 (SDA/GPIO2)
- net at J6.1 (3V3), J6.17 (3V3): now also R18.1
- new net: LED5.2 (A), R18.2
- no-connect marks 0 -> 116
Other:
- sheet RF_TRANSMITTER ports: added RF_TRANSMITER_EN; removed none
- sheet acc-gyr ports: added none; removed AD0/SDO
- sheet motor_driver ports: added none; removed ENC_A, ENC_B
- sheet motor_driver1 ports: added none; removed ENC_A, ENC_B
- sheet motor_driver2 ports: added none; removed ENC_A, ENC_B
- sheet motor_driver3 ports: added none; removed ENC_A, ENC_B
- sheet motor_driver4 ports: added none; removed ENC_A, ENC_B
- sheet motor_driver5 ports: added none; removed ENC_A, ENC_B
- sheet motor_driver6 ports: added none; removed ENC_A, ENC_B
- sheet motor_driver7 ports: added none; removed ENC_A, ENC_B
- sheet motor_driver8 ports: added none; removed ENC_A, ENC_B
- sheet motor_driver9 ports: added none; removed ENC_A, ENC_B
- moved on the sheet: J12
